File: Hardware/InkTime.sch (EAGLE design)
At the start: 123 parts, among them IC1 BQ25180, IC2 DRV2605, IC3 BMA423, IC9 RT6160, J1 EPD FPC 24pin, J2 TC2030-IDC, J4 USB-C, Q1 DMG2305, Q3 SI1308, U1 nRF52840, U3 MAX17048, X1 32MHz, X2 32.768kHz

Commit message: Update 1
Parts:
- removed C26: 10uF, InkTime_v5:PERFECT_0402_CAP_0402
- removed C28: 4.7uF, InkTime_v5:PERFECT_0402_CAP_0402
- removed C35, C36: 1uF/50V, InkTime_v5:ESP32_C6_LIBRARY_1_ESP32_WROVER_EAGLE-LTSPICE_CC0402
- removed FRAME1: InkTime - MCU/Power/IMU/SWD, InkTime_v5:FRAMES_A3L-LOC
- removed FRAME2: InkTime - EPD/Peripherals, InkTime_v5:FRAMES_A3L-LOC
- removed GND1, GND10, GND11, GND12, GND13, GND14, GND15, GND16, GND17, GND18, GND19, GND2, GND20, GND21, GND22, GND23, GND24, GND25, GND26, GND27, GND28, GND29, GND3, GND30, GND4, GND5, GND6, GND7, GND8, GND9: SUPPLY1_GND, InkTime_v5:SUPPLY1_GND
- removed R1, R15, R19: 10K, InkTime_v5:CPF0201D7K68C1_CPF0201D7K68C1
- removed R10, R11, R16, R6: 100K, InkTime_v5:CPF0201D7K68C1_CPF0201D7K68C1
- removed R12: 3K3, InkTime_v5:CPF0201D7K68C1_CPF0201D7K68C1
- removed R13, R14: 1M, InkTime_v5:CPF0201D7K68C1_CPF0201D7K68C1
- removed R20: 47K, InkTime_v5:CPF0201D7K68C1_CPF0201D7K68C1
- removed TP1: SWO, InkTime_v5:HECTOR_WATCH_1_TPTP20R
- removed TP2: SWDCLK, InkTime_v5:HECTOR_WATCH_1_TPTP20R
- removed TP3: SWDIO, InkTime_v5:HECTOR_WATCH_1_TPTP20R
- removed TP4: RESET, InkTime_v5:HECTOR_WATCH_1_TPTP20R
- removed TP5: VBAT, InkTime_v5:HECTOR_WATCH_1_TPTP20R
- removed TP6: 3V3, InkTime_v5:HECTOR_WATCH_1_TPTP20R
- removed TP7: GND, InkTime_v5:HECTOR_WATCH_1_TPTP20R
- added C1-EP-DR: 10uF, InkTime_v5:NORDIC_NRF_3_CAPACITOR_0402_N
- added C2-EP-DR: 4.7uF/25V, InkTime_v5:NORDIC_NRF_3_CAPACITOR_0402_N
- added C38: 1uF/16V, InkTime_v5:NORDIC_NRF_3_CAPACITOR_0402_N
- added C39: 10uF/16V, InkTime_v5:NORDIC_NRF_3_CAPACITOR_0402_N
- added C42: 0.1uF/16V, InkTime_v5:NORDIC_NRF_3_CAPACITOR_0201_N
- added C43: 4.7uF/16V, InkTime_v5:NORDIC_NRF_3_CAPACITOR_0402_N
- added C_RESET: 100nF/10V, InkTime_v5:NORDIC_NRF_3_CAPACITOR_0201_N
- added D_TVS: MBR0530 (TVS clamp), InkTime_v5:ESP32_C6_LIBRARY_5_MBR0530
- added EPD_C1, EPD_C10, EPD_C11, EPD_C12, EPD_C2, EPD_C6, EPD_C7, EPD_C8, EPD_C9: 1uF/50V, InkTime_v5:NORDIC_NRF_3_CAPACITOR_0402_N
- added EPD_C5: 0.1uF/50V, InkTime_v5:NORDIC_NRF_3_CAPACITOR_0402_N
- added F1: 0R (FUSE), InkTime_v5:CPF0201D7K68C1_CPF0201D7K68C1
- added R1_EP_DR: 0.47, InkTime_v5:CPF0201D7K68C1_CPF0201D7K68C1
- added R1_USB, R2_USB: 5K1, InkTime_v5:CPF0201D7K68C1_CPF0201D7K68C1
- added R2_EP_DR, R_PWR_EPD, R_RESET: 10K, InkTime_v5:CPF0201D7K68C1_CPF0201D7K68C1
- added R_ALERT, R_PMIC_INT: 100K, InkTime_v5:CPF0201D7K68C1_CPF0201D7K68C1
- added R_TYPE_SEL: 2.2, InkTime_v5:CPF0201D7K68C1_CPF0201D7K68C1
- added TP_3.3V, TP_3V3, TP_BAT_GND, TP_GND, TP_ON, TP_OP, TP_RESET, TP_SCL, TP_SDA, TP_SWDCLK, TP_SWDIO, TP_SWO, TP_VBAT, TP_VBUS, TP_VREG: HECTOR_WATCH_1_TPTP20R, InkTime_v5:HECTOR_WATCH_1_TPTP20R
- ANT1: value 2450AT18B100 -> 2450AT18B100E; device InkTime_v5:2450AT18B100E_2450AT18B100E -> InkTime_v5:2450AT18B100E_2450AT18B100E3D
- C1, C17, C18, C2: value 12pF -> 12pF/10V; device InkTime_v5:NORDIC_NRF_3_CAPACITOR_0201_L -> InkTime_v5:NORDIC_NRF_3_CAPACITOR_0201_N
- C10, C13, C22: value 100nF -> N.C.; device InkTime_v5:NORDIC_NRF_3_CAPACITOR_0201_L -> InkTime_v5:NORDIC_NRF_3_CAPACITOR_0201_N
- C11: value 100nF -> 100pF/10V; device InkTime_v5:NORDIC_NRF_3_CAPACITOR_0201_L -> InkTime_v5:NORDIC_NRF_3_CAPACITOR_0201_N
- C12, C19, C5, C7, C8: value 100nF -> 100nF/10V; device InkTime_v5:NORDIC_NRF_3_CAPACITOR_0201_L -> InkTime_v5:NORDIC_NRF_3_CAPACITOR_0201_N
- C14, C6: value 4.7uF -> 4.7uF/10V; device InkTime_v5:PERFECT_0402_CAP_0402 -> InkTime_v5:NORDIC_NRF_3_CAPACITOR_0402_N
- C15: value 10uF -> 1uF/10V; device InkTime_v5:PERFECT_0402_CAP_0402 -> InkTime_v5:NORDIC_NRF_3_CAPACITOR_0402_N
- C16: value 47nF -> 47nF/10V; device InkTime_v5:NORDIC_NRF_3_CAPACITOR_0201_L -> InkTime_v5:NORDIC_NRF_3_CAPACITOR_0201_N
- C20, C21: value 100nF -> 4.7uF/10V; device InkTime_v5:NORDIC_NRF_3_CAPACITOR_0201_L -> InkTime_v5:NORDIC_NRF_3_CAPACITOR_0402_N
- C23: value 100nF -> 0.1uF/10V; device InkTime_v5:NORDIC_NRF_3_CAPACITOR_0201_L -> InkTime_v5:NORDIC_NRF_3_CAPACITOR_0201_N
- C24: value 47nF -> 10uF/10V; device InkTime_v5:NORDIC_NRF_3_CAPACITOR_0201_L -> InkTime_v5:NORDIC_NRF_3_CAPACITOR_0402_N
- C25: value 10uF -> 22uF/10V; device InkTime_v5:PERFECT_0402_CAP_0402 -> InkTime_v5:NORDIC_NRF_3_CAPACITOR_0402_N
- C27: value 10uF -> 0.1uF/10V; device InkTime_v5:PERFECT_0402_CAP_0402 -> InkTime_v5:NORDIC_NRF_3_CAPACITOR_0201_N
- C29, C30, C31: value 1uF -> 1uF/10V; device InkTime_v5:PERFECT_0402_CAP_0402 -> InkTime_v5:NORDIC_NRF_3_CAPACITOR_0402_N
- C3: value 0.8pF -> 1pF/10V; device InkTime_v5:NORDIC_NRF_3_CAPACITOR_0201_L -> InkTime_v5:NORDIC_NRF_3_CAPACITOR_0201_N
- C32: value 1uF -> 0.1uF/10V; device InkTime_v5:PERFECT_0402_CAP_0402 -> InkTime_v5:NORDIC_NRF_3_CAPACITOR_0201_N
- C33: value 4.7uF -> 22uF/10V; device InkTime_v5:PERFECT_0402_CAP_0402 -> InkTime_v5:NORDIC_NRF_3_CAPACITOR_0402_N
- C34: value 1uF/50V -> 0.1uF/10V; device InkTime_v5:ESP32_C6_LIBRARY_1_ESP32_WROVER_EAGLE-LTSPICE_CC0402 -> InkTime_v5:NORDIC_NRF_3_CAPACITOR_0201_N
- C37: value 1uF/50V -> 1uF/16V; device InkTime_v5:ESP32_C6_LIBRARY_1_ESP32_WROVER_EAGLE-LTSPICE_CC0402 -> InkTime_v5:NORDIC_NRF_3_CAPACITOR_0402_N
- C4: value 0.5pF -> 1pF/10V; device InkTime_v5:NORDIC_NRF_3_CAPACITOR_0201_L -> InkTime_v5:NORDIC_NRF_3_CAPACITOR_0201_N
- C9: value 1pF -> 820pF/10V N.C.; device InkTime_v5:NORDIC_NRF_3_CAPACITOR_0201_L -> InkTime_v5:NORDIC_NRF_3_CAPACITOR_0201_N
- IC1: value BQ25180 -> BQ25180YBGR
- IC2: value DRV2605 -> DRV2605YZFR
- IC3: value BMA423 -> BMA421; device InkTime_v5:BMA423_BMA423 -> InkTime_v5:BMA421_BMA421
- IC9: value RT6160 -> RT6160AWSC
- J1: value EPD FPC 24pin -> 503480-2400; device InkTime_v5:503480-2400_503480-2400 -> InkTime_v5:503480-2400_503480-24003D
- J4: value USB-C -> KH-TYPE-C-16P
- L1: device InkTime_v5:NORDIC_NRF_2_INDUCTOR_0201_L -> InkTime_v5:NORDIC_NRF_2_INDUCTOR_0402_N
- L2: value 15nH -> 10uH; device InkTime_v5:NORDIC_NRF_2_INDUCTOR_0201_L -> InkTime_v5:NORDIC_NRF_2_INDUCTOR_0603_N
- L3: value 10uH -> 15nH; device InkTime_v5:NORDIC_NRF_2_INDUCTOR_0402_L -> InkTime_v5:NORDIC_NRF_2_INDUCTOR_0402_N
- L7: value 4.7uH -> FTC252012SR47MBCA
- Q1: value DMG2305 -> 20V/4.2A/52mΩ/1.4W
- Q3: value SI1308 -> SI1308EDL-T1-GE3
- R17, R18: value 4K7 -> 3K3
- R2: value 10K -> 0
- R3, R4: value 5.1K -> 0
- SJ1: value SJ -> (none)
- SW_DN, SW_ENT, SW_UP: value EVP-AKE31A -> 2025-10-22_07-23-44_LIBRARY_EVP-AKE31ASW_EVP-AKE31A_PAN
- U1: value nRF52840 -> NRF52840_QF; device InkTime_v5:NORDIC_NRF_4_NRF52840_QF -> InkTime_v5:NORDIC_NRF_4_NRF52840_QF_PINCLEAN
- U3: value MAX17048 -> MAX17048G+T10
- X1: value 32MHz -> 32MHz ±10ppm
- X2: value 32.768kHz -> 32.768kHz ±20ppm
Connections:
- net DEC1 renamed N$112
- removed net CC1: J4.CC1, R3.1
- removed net CC2: J4.CC2, R4.1
- removed net D+: D3.I/O1_1, D3.I/O1_2, J4.DP1, J4.DP2, U1.D+@AD6
- removed net D-: D3.I/O2_1, D3.I/O2_2, J4.DN1, J4.DN2, U1.D-@AD4
- removed net DCC: C15.1, L3.1, U1.DCC@B3
- removed net DCCH: C16.1, L3.2, U1.DCCH@AB2
- removed net DEC3V3: C19.1, U1.DEC3V3@AC5
- removed net EPD_EN: Q1.G, R10.2, R11.1
- removed net N$1: C3.1, L1.2, L2.1
- removed net N$10: D2.A, L5.2
- removed net N$11: D4.A
- removed net N$12: C36.1, D5.K
- removed net N$2: ANT1.FEED, C4.1, L2.2
- removed net N$20: SJ1.1
- removed net N$21: SJ1.2
- removed net N$3: IC3.SDO, R1.2
- removed net N$4: IC2.REG, R12.2
- removed net N$5: U3.QSTRT
- removed net N$6: U3.CTG
- removed net SW_DN_NET: C30.1, R7.2, SW_DN.1, U1.P1.04@U24
- removed net SW_ENT_NET: C31.1, R8.2, SW_ENT.1, U1.P1.05@T23
- removed net SW_UP_NET: C29.1, R5.2, SW_UP.1, U1.P1.03@V23
- removed net VDDH: C20.1, U1.VDDH@Y2
- removed net XL1: C17.1, U1.P0.00/XL1@D2, X2.1
- removed net XL2: C18.1, U1.P0.01/XL2@F2, X2.2
- new net DN: D3.I/O1_1, J4.DN1, J4.DN2
- new net DP: D3.I/O2_1, J4.DP1, J4.DP2
- new net D_N: D3.I/O1_2, U1.D-@AD4
- new net D_P: D3.I/O2_2, U1.D+@AD6
- new net N$101: L2.1, L3.2
- new net N$102: L2.2, U1.DCC@B3
- new net N$103: IC1.TS/MR, R9.2
- new net N$104: C3.1, L1.1, U1.ANT@H23
- new net N$105: J4.CC1, R1_USB.2
- new net N$107: C9.1, U1.DEC5@N24
- new net N$111: C17.2, U1.P0.00/XL1@D2, X2.2
- new net N$113: EPD_C2.2, J1.4
- new net N$114: R1_EP_DR.1, R_TYPE_SEL.2, SJ1.2
- new net N$115: IC9.SDA, R2.2
- new net N$116: EPD_C1.2, J1.5
- new net N$117: C20.1, U1.DEC3V3@AC5
- new net N$118: IC9.SCL, R4.2
- new net N$119: IC3.SDO, R3.2
- new net N$120: C18.2, U1.P0.01/XL2@F2, X2.1
- new net N$121: C2-EP-DR.2, D5.A, L5.1, Q3.D
- new net N$122: C13.1, U1.DEC2@A18
- new net N$123: C32.1, IC2.REG
- new net N$126: C2-EP-DR.1, D2.K, D4.A
- new net N$131: J4.CC2, R2_USB.1
- new net N$134: EPD_C6.2, J1.18
- new net N$136: EPD_C7.2, J1.19
- new net N$137: EPD_C8.2, J1.20
- new net N$141: EPD_C10.2, J1.22
- new net N$145: EPD_C12.2, J1.24
- new net P0.09: U1.P0.09/NFC1@L24
- new net P0.13: C30.1, R5.1, SW_UP.2, U1.P0.13@AD8
- new net P0.14: C31.1, R8.1, SW_ENT.2, U1.P0.14@AC9
- new net P0.20: U1.P0.20@AD16
- new net P0.21: U1.P0.21@AC17
- new net P0.22: U1.P0.22@AD18
- new net P0.23: U1.P0.23@AC19
- new net P0.24: U1.P0.24@AD20
- new net P0.25: U1.P0.25@AC21
- new net P0.26: U1.P0.26@G1
- new net P0.27: U1.P0.27@H2
- new net P0.28: U1.P0.28/AIN4@B11
- new net P0.30: U1.P0.30/AIN6@B9
- new net P1.01: Q1.G, R_PWR_EPD.1, U1.P1.01@Y23
- new net P1.02: C29.1, R7.1, SW_DN.2, U1.P1.02@W24
- new net P1.03: U1.P1.03@V23
- new net P1.04: U1.P1.04@U24
- new net P1.05: U1.P1.05@T23
- new net P1.06: U1.P1.06@R24
- new net P1.07: U1.P1.07@P23
- new net P1.10: U1.P1.10@A20
- new net P1.11: U1.P1.11@B19
- new net P1.12: U1.P1.12@B17
- new net P1.13: U1.P1.13@A16
- new net P1.14: U1.P1.14@B15
- new net P1.15: U1.P1.15@A14
- net 3V3: now also C12.1, C14.1, C19.1, C25.1, C34.1, C6.1, IC3.CSB, J2.1, Q1.S, R5.2, R7.2, R8.2, R_ALERT.2, R_PMIC_INT.2, R_PWR_EPD.2, R_RESET.2, TP_3.3V.TP, TP_3V3.TP, U1.VDDH@Y2; no longer C21.1, C22.1, C27.1, C28.1, C32.1, Q1.D, R10.1, R15.1, R5.1, R7.1, R8.1, TP6.TP, U3.VDD
- net ALERT: now also R_ALERT.1, U1.P0.10/NFC2@J24; no longer U1.P0.16@AC11
- net DEC3: now also C11.1; no longer C14.1
- net DEC4_6: now also C10.1, C15.1, C16.1, L3.1; no longer C6.1, U1.DEC5@N24
- net EPD_3V3: now also C1-EP-DR.1, EPD_C5.2, J1.15, J1.16, L5.2, Q1.D; no longer C10.1, C11.1, C12.1, C13.1, C23.1, Q1.S
- net EPD_BUSY: now also J1.9, U1.P0.17@AD12; no longer J1.11, U1.P0.05/AIN3@K2
- net EPD_CS: now also J1.12, U1.P0.05/AIN3@K2; no longer J1.6, U1.P0.07@M2
- net EPD_DC: now also J1.11, U1.P0.15@AD10; no longer J1.9, U1.P0.06@L1
- net EPD_RST: now also U1.P0.16@AC11; no longer U1.P0.15@AD10
- net GDR: now also Q3.G, R2_EP_DR.2; no longer L5.1
- net GND: now also C1-EP-DR.2, C14.2, C15.2, C16.2, C17.1, C18.1, C19.2, C2.2, C20.2, C23.1, C24.1, C38.2, C39.2, C42.2, C43.2, C5.2, C6.2, C7.2, C8.2, C_RESET.2, D4.K, D_TVS.A, EPD_C1.1, EPD_C10.1, EPD_C11.1, EPD_C12.1, EPD_C2.1, EPD_C5.1, EPD_C6.1, EPD_C7.1, EPD_C8.1, EPD_C9.1, IC2.IN/TRIG, IC9.VSEL, J1.17, J1.8, R1_USB.1, R2_EP_DR.1, R2_USB.2, R3.1, R9.1, R_TYPE_SEL.1, SJ1.1, SW_DN.1, SW_ENT.1, SW_UP.1, TP_BAT_GND.TP, TP_GND.TP, U3.CTG, U3.QSTRT, X1.2, X1.4; no longer C18.2, C23.2, C26.2, C28.2, C35.2, C36.2, GND1.GND, GND10.GND, GND11.GND, GND12.GND, GND13.GND, GND14.GND, GND15.GND, GND16.GND, GND17.GND, GND18.GND, GND19.GND, GND2.GND, GND20.GND, GND21.GND, GND22.GND, GND23.GND, GND24.GND, GND25.GND, GND26.GND, GND27.GND, GND28.GND, GND29.GND, GND3.GND, GND30.GND, GND4.GND, GND5.GND, GND6.GND, GND7.GND, GND8.GND, GND9.GND, Q1.S, Q3.S, SW_DN.2, SW_ENT.2, SW_UP.2, TP7.TP
- net IMU_INT1: now also U1.P0.08@N1; no longer U1.P1.08@P2
- net IMU_INT2: now also U1.P1.08@P2; no longer U1.P0.11@T2
- net MOSI: now also J1.14, U1.P0.03/AIN1@B13; no longer J1.7, U1.P0.13@AD8
- net OUT+: now also TP_OP.TP
- net OUT-: now also TP_ON.TP
- net PMIC_INT: now also R_PMIC_INT.1, U1.P0.11@T2; no longer U1.P0.08@N1
- net PREVGH: now also D5.K, EPD_C9.2, J1.21; no longer C34.1, D2.K, J1.4
- net PREVGL: now also D2.A, EPD_C11.2, J1.23; no longer C35.1, D4.K, J1.3
- net RESE: now also J1.3, Q3.S, R1_EP_DR.2; no longer J1.5, R16.1
- net RESET: now also C_RESET.1, R_RESET.1, TP_RESET.TP, U1.P0.19@AC15; no longer R15.2, TP4.TP
- net RF: now also ANT1.FEED, C22.1, C4.1, L1.2; no longer C9.1, L1.1, U1.ANT@H23
- net SCK: now also J1.13, U1.P0.02/AIN0@A12; no longer J1.8, U1.P0.14@AC9
- net SCL: now also IC3.SCX, R4.1, TP_SCL.TP, U1.P0.07@M2; no longer IC3.ASCL, IC9.SCL, U1.P0.26@G1
- net SDA: now also IC3.SDX, R2.1, TP_SDA.TP, U1.P0.06@L1; no longer IC3.ASDA, IC9.SDA, U1.P0.27@H2
- net SWDCLK: now also TP_SWDCLK.TP; no longer TP2.TP
- net SWDIO: now also TP_SWDIO.TP; no longer TP3.TP
- net SWO: now also TP_SWO.TP, U1.P1.00@AD22; no longer TP1.TP, U1.P1.09@R1
- net VBAT: now also C27.1, C37.1, TP_VBAT.TP, U3.VDD; no longer TP5.TP
- net VBUS: now also C21.1, C38.1, C42.1, C43.1, D_TVS.K, F1.1, F1.2, TP_VBUS.TP; no longer C25.1
- net VREG: now also C23.2, C24.2, C39.1, TP_VREG.TP; no longer C26.1, R6.1
- net XC2: now also X1.3; no longer X1.2
Other:
- note added: "DC/DC"
- note added: "E-Paper Display Connector"
- note added: "E-Paper Drive Circuit"
- note added: "Fuel Gauge"
- note added: "Haptic Driver"
- note added: "IMU"
- note added: "LiPo Charger"
- note added: "SWD"
- note added: "USB C Connector & ESD Protection"
- note removed: "E-Paper Display FPC Connector"
- note removed: "EPD Drive Circuit"
- note removed: "EPD Power (MOSFET switch & boost)"
- note removed: "Fuel Gauge / Haptic Driver"
- note removed: "IMU (BMA423)"
- note removed: "InkTime Smartwatch - Sheet 1: MCU / Power / IMU / SWD"
- note removed: "InkTime Smartwatch - Sheet 2: EPD / Peripherals"
- note removed: "Power Management"
- note removed: "RF Matching Network & Antenna"
- note removed: "SWD Debug / Test Points"
- note removed: "Solder Jumper / Misc"
- note removed: "nRF52840 SoC"
